File: 002-main/002-main.brd (EAGLE design)
At the start: 106 x 53 mm, 78 parts, among them IC1 MEGA8-AI, J1 22057045, J2 22057045, J3 22057035, J4 22057035, J5 22057035, J6 22057035, J7 22057035, J8 5267-5, J9 5267-4, Q1 C1015, U1 CH340ESMD, U2 STM32F446RET6, U3 CH340ESMD, U5 MAX485ESA+T, X1 Seeed Studio XIAO ESP32C3, Y1 16MHz

Commit message: ATmega消す
Parts:
- added C16, C17: 0.1µ, rcl:C0603
- added R18, R19: 100, rcl:R0402
- added U6: HX711, HX711:SOP127P600X180-16N
Connections:
- new net L-EXC+: U6.3
- new net L-INA+: R19.2
- new net L-INA-: R18.2
- new net N$29: C16.1, R18.1, U6.7
- new net N$30: C16.2, R19.1, U6.8
- new net N$31: C17.1, U6.6
- net +5V: now also U6.1, U6.16
- net GND: now also C17.2, U6.5

Commit message: ほぼ完了
Parts:
- removed C17: 0.1µ, rcl:C0603
- removed LED17, LED19: WHITE, led:SML0603
- removed U3: CH340ESMD, CH340E:MSOP10
- removed U6: HX711, HX711:SOP127P600X180-16N
- removed X4: (no value), microbuilder:USB_C_CUSB31-CFM2AX-01-X
- removed Y1: 16MHz, 7325-0800A2010-00:O3225100MEDA4SC
- added IC2: NJU77551F, burr-brown:SOT23-5
- added J10, J11, J12: 22057045, con-molex-5268:CON_22057045_MOL
- added J13: 5267-4, con-molex-spox:5267-4
- added JP2: JP2, jp:JP2
- added LS1: MLT-8530, MLT-8530:MLT-8530_JHE
- added R20, R21, R24, R25: 330k, rcl:R0402
- added R22, R23, R26, R27, R28, R29: 1k, rcl:R0402
- added R30, R31: 10k, rcl:R0402
- added S1: (no value), switch-omron:B3F-31XX
- added SW1: SK-12D11VG3, Slide Switch:SK-12D11VG3
- added T1, T2, T3: BSS138, zetex:SOT-23
- C15: value 0.1µ -> 100μ; device rcl:C0603 -> rcl:153CLV-0505
- IC1: value MEGA8-AI -> NJU77551F; device atmel:TQFP32-08 -> burr-brown:SOT23-5
- J9: value 5267-4 -> 22057045; device con-molex-spox:5267-4 -> con-molex-5268:CON_22057045_MOL
- JP1: value (none) -> JP2; device pinhead:1X04/90 -> jp:JP2
- R11: value 270 -> 180k
- R18, R19: value 100 -> 1k
- R4, R5: value 5k1 -> 10k
- R6: value 270 -> 10k
- moved R19 99.4 mm to (24.7, 45.1)
- moved R18 96.4 mm to (24.7, 44.0)
- moved C16 85.2 mm to (-1.00, 50.0), turned to 90 degrees
- moved R5 81.5 mm to (37.5, 37.0), turned to 270 degrees
- moved R4 75.5 mm to (39.0, 37.0), turned to 270 degrees
- moved R6 71.7 mm to (36.0, 37.0), turned to 270 degrees
- moved IC1 48.8 mm to (21.4, 44.0), turned to 270 degrees
- moved R13 40.5 mm to (-27.0, 30.5)
- moved R12 36.4 mm to (-27.0, 31.6)
- moved U4 35.9 mm to (-19.1, 23.7), turned to 180 degrees
- moved X1 28.2 mm to (10.0, 49.0), turned to 0 degrees
- moved JP1 19.2 mm to (-27.9, 39.4), turned to 90 degrees
- moved LED14 18.0 mm to (51.0, 13.5), turned to 270 degrees
- moved LED8 18.0 mm to (51.0, 31.5), turned to 270 degrees
- moved C15 16.4 mm to (-31.6, 19.2), turned to 270 degrees
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Connections:
- removed net AVCC: IC1.18
- removed net AVR-CTS: U3.5
- removed net AVR-D+: U3.1, X4.A6, X4.B6
- removed net AVR-D-: U3.2, X4.A7, X4.B7
- removed net AVR-RTS: U3.4
- removed net AVR-RX: IC1.30, U3.8
- removed net AVR-TX: IC1.31, U3.9
- removed net L-EXC+: U6.3
- removed net L-INA+: R19.2
- removed net L-INA-: R18.2
- removed net N$31: C17.1, U6.6
- removed net OSC1: IC1.7, Y1.1
- removed net OSC2: IC1.8, Y1.3
- new net LCELL-L: IC1.1, R21.1
- new net LCELL-R: IC2.1, R25.1
- new net LED-FLOOR: J11.4
- new net LED-L-5V: JP1.2, LED1.3, R26.2, T2.1
- new net LED-R-5V: JP2.2, LED8.3, R28.2, T3.1
- new net SIG-FLOOR: J11.3, R11.2
- new net SPK: T1.3
- net +3V3: now also IC1.5, IC2.5, J10.1, J12.1, LS1.1, R27.1, R29.1, R30.1, R4.1, R5.1, R6.1, SW1.3, T2.3, T3.3
- net +5V: now also J11.1, R11.1, R26.1, R28.1; no longer IC1.4, IC1.6, U3.7, U6.1, U6.16
- net BOOT0: now also R31.1, SW1.1
- net GND: now also C15.-, C16.2, IC1.2, IC2.2, J10.2, J11.2, J12.2, J13.P$4, R20.1, R24.1, R31.2, S1.2, SW1.4, SW1.5, T1.2; no longer C15.2, C17.2, IC1.21, IC1.3, IC1.5, JP1.4, LED19.C, R4.2, R5.2, R6.1, U3.3, U6.5, X4.A1B12, X4.B1A12, Y1.2, Y1.4
- net LED-L: now also JP1.1, R27.2, T2.2; no longer LED1.3
- net LED-R: now also JP2.1, R29.2, T3.2; no longer LED8.3
- net LED-UI: now also J9.4; no longer J9.P$4
- net N$17: now also LS1.2, T1.1; no longer R4.1, X4.A5
- net N$19: now also IC1.3, R18.1, R20.2; no longer R5.1, X4.B5
- net N$20: now also IC1.4, R19.1, R21.2; no longer LED17.A, X4.A4B9, X4.B4A9
- net N$21: now also J10.3, R19.2; no longer LED17.C, R6.2
- net N$24: now also J10.4, R18.2; no longer C15.1, U3.10
- net N$25: now also IC2.3, R22.1, R24.2; no longer R11.2, U3.6
- net N$26: now also IC2.4, R23.1, R25.2; no longer LED19.A, R11.1
- net N$29: now also J12.4, R22.2; no longer C16.1, R18.1, U6.7
- net N$30: now also J12.3, R23.2; no longer C16.2, R19.1, U6.8
- net NRST: now also C16.1, J13.P$3, R30.2, S1.1; no longer JP1.3
- net SW1: now also J9.3, R6.2; no longer J9.P$3
- net SW2: now also J9.2, R5.2; no longer J9.P$2
- net SWCLK: now also J13.P$1; no longer JP1.1
- net SWDIO: now also J13.P$2; no longer JP1.2
- net TOGGLE: now also J9.1, R4.2; no longer J9.P$1
- net VDD: now also C15.+
Routing:
- net +3V3: track 41.3 -> 225.9 mm, vias 0 -> 15
- net +5V: track 159.2 -> 290.4 mm, vias 6 -> 8
- net GND: track 983.9 -> 1085.3 mm, vias 40 -> 43
- net NRST: track 0.00 -> 66.0 mm, vias 0 -> 2
- net LED-L-5V: track 0.00 -> 35.1 mm, vias 0 -> 2
- net LED-R-5V: track 0.00 -> 30.6 mm
- net UART3-TX: track 54.1 -> 27.8 mm
- net UART3-RX: track 36.4 -> 10.6 mm
- net BOOT0: track 0.00 -> 25.1 mm, vias 0 -> 2
- net SWDIO: track 8.07 -> 25.8 mm, vias 1 -> 0
- net N$21: track 1.58 -> 18.3 mm
- net SCL: track 33.0 -> 18.1 mm, vias 0 -> 1
- net N$24: track 5.67 -> 18.4 mm
- net SDA: track 30.0 -> 20.6 mm, vias 0 -> 1
- net AVR-RX: track 9.27 -> 0.00 mm
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Other:
- outline, holes or cut-outs redrawn
- board text added: "+"
- board text removed: "USB-SIGNAL"
