File: 002-main/002-main.sch (EAGLE design)
At the start: 83 parts, among them IC1 MEGA8-AI, J1 22057045, J2 22057045, J3 22057035, J4 22057035, J5 22057035, J6 22057035, J7 22057035, J8 5267-5, J9 5267-4, Q1 C1015, U1 CH340ESMD, U2 STM32F446RET6, U3 CH340ESMD, U5 MAX485ESA+T, U6 HX711, X1 Seeed Studio XIAO ESP32C3, Y1 16MHz

Commit message: ほぼ完了
Parts:
- removed C17: 0.1µ, rcl:C-EUC0603
- removed LED17, LED19: WHITE, led:LEDSML0603
- removed U3: CH340ESMD, CH340E:CH340ESMD
- removed U6: HX711, HX711:HX711
- removed X4: (no value), microbuilder:USB_C
- removed Y1: 16MHz, 7325-0800A2010-00:O3225100MEDA4SC
- added IC2: NJU77551F, burr-brown:OPA340N
- added J10, J11, J12: 22057045, con-molex-5268:22057045
- added J13: 5267-4, con-molex-spox:5267-4
- added JP2: JP2, jp:JP2
- added LS1: MLT-8530, MLT-8530:MLT-8530
- added R20, R21, R24, R25: 330k, rcl:R-EU_R0402
- added R22, R23, R26, R27, R28, R29: 1k, rcl:R-EU_R0402
- added R30, R31: 10k, rcl:R-EU_R0402
- added S1: (no value), switch-omron:31-XX
- added SW1: SK-12D11VG3, Slide Switch:SK-12D11VG3
- added T1, T2, T3: BSS138, zetex:NMOSSOT23
- C15: value 0.1µ -> 100μ; device rcl:C-EUC0603 -> rcl:CPOL-EU153CLV-0505
- IC1: value MEGA8-AI -> NJU77551F; device atmel:MEGA8-AI -> burr-brown:OPA340N
- J9: value 5267-4 -> 22057045; device con-molex-spox:5267-4 -> con-molex-5268:22057045
- JP1: value (none) -> JP2; device pinhead:PINHD-1X4/90 -> jp:JP2
- R11: value 270 -> 180k
- R18, R19: value 100 -> 1k
- R4, R5: value 5k1 -> 10k
- R6: value 270 -> 10k
Connections:
- removed net AVR-CTS: U3.CTS
- removed net AVR-D+: U3.UD+, X4.D+
- removed net AVR-D-: U3.UD-, X4.D-
- removed net AVR-RTS: U3.RTS
- removed net AVR-RX: IC1.PD0(RXD), U3.TX
- removed net AVR-TX: IC1.PD1(TXD), U3.RX
- removed net L-EXC+: U6.AVDD
- removed net L-INA+: R19.2
- removed net L-INA-: R18.2
- removed net N$31: C17.1, U6.VBG
- removed net OSC1: IC1.PB6(XTAL1/TOSC1), Y1.E/D
- removed net OSC2: IC1.PB7(XTAL2/TOSC2), Y1.OUTPUT
- new net LCELL-L: IC1.OUT, R21.1
- new net LCELL-R: IC2.OUT, R25.1
- new net LED-FLOOR: J11.4
- new net LED-L-5V: JP1.2, LED1.DI, R26.2, T2.D
- new net LED-R-5V: JP2.2, LED8.DI, R28.2, T3.D
- new net SIG-FLOOR: J11.3, R11.2
- new net SPK: T1.G
- net +3V3: now also IC1.V+, IC2.V+, J10.1, J12.1, LS1.1, R27.1, R29.1, R30.1, R4.1, R5.1, R6.1, SW1.O, T2.G, T3.G
- net +5V: now also J11.1, R11.1, R26.1, R28.1; no longer IC1.VCC@1, IC1.VCC@2, U3.VCC, U6.DVDD, U6.VSUP
- net BOOT0: now also R31.1, SW1.P
- net GND: now also C15.-, C16.2, IC1.V-, IC2.V-, J10.2, J11.2, J12.2, J13.-4, R20.1, R24.1, R31.2, S1.S, SW1.CASE, T1.S; no longer C15.2, C17.2, IC1.GND, IC1.GND@1, IC1.GND@2, JP1.4, LED19.C, R4.2, R5.2, R6.1, U3.GND, U6.AGND, X4.GND, Y1.GND, Y1.VDD
- net LED-L: now also JP1.1, R27.2, T2.S; no longer LED1.DI
- net LED-R: now also JP2.1, R29.2, T3.S; no longer LED8.DI
- net LED-UI: now also J9.4; no longer J9.-4
- net N$17: now also LS1.2, T1.D; no longer R4.1, X4.CC1
- net N$19: now also IC1.+IN, R18.1, R20.2; no longer R5.1, X4.CC2
- net N$20: now also IC1.-IN, R19.1, R21.2; no longer LED17.A, X4.VBUS
- net N$21: now also J10.3, R19.2; no longer LED17.C, R6.2
- net N$24: now also J10.4, R18.2; no longer C15.1, U3.V3
- net N$25: now also IC2.+IN, R22.1, R24.2; no longer R11.2, U3.TNOW
- net N$26: now also IC2.-IN, R23.1, R25.2; no longer LED19.A, R11.1
- net N$29: now also J12.4, R22.2; no longer C16.1, R18.1, U6.INA-
- net N$30: now also J12.3, R23.2; no longer C16.2, R19.1, U6.INA+
- net NRST: now also C16.1, J13.-3, R30.2, S1.P; no longer JP1.3
- net SW1: now also J9.3, R6.2; no longer J9.-3
- net SW2: now also J9.2, R5.2; no longer J9.-2
- net SWCLK: now also J13.-1; no longer JP1.1
- net SWDIO: now also J13.-2; no longer JP1.2
- net TOGGLE: now also J9.1, R4.2; no longer J9.-1
- net VDD: now also C15.+
Other:
- note added: "BOOT0"
- note added: "FLOOR"
- note added: "LOAD CELL"
- note added: "Logic Level Converter"
- note added: "Pull-up"
- note added: "RESET"
- note added: "SPK"
- note added: "UI"
- moved on the sheet: C16, C7, C8, C9, D1, R11, R18, R19, R4, R5, R6, REG1

Commit message: ひとまず完了
Parts:
- added D3: 1N4001, diode:GF1
Connections:
- new net N$31: D3.C, X1.5V
- net +5V: now also D3.A
- net LED-FLOOR: now also U2A.PB15
- net LED-L: now also U2A.PA15
- net LED-R: now also U2A.PB13
- net LED-UI: now also U2A.PB14
- net SIG-FLOOR: now also U2A.PC0
- net SW1: now also U2A.PA4
- net SW2: now also U2A.PA5
- net TOGGLE: now also U2A.PA6
Changed lines of the file:
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@@
 </variantdefs>
 <classes>
-<class number="0" name="default" width="0" drill="0">
+<class number="0" name="default" width="0.127" drill="0">
 </class>
 </classes>
@@
 <part name="GND60" library="supply1" library_urn="urn:adsk.eagle:library:371" deviceset="GND" device=""/>
 <part name="+3V16" library="supply1" library_urn="urn:adsk.eagle:library:371" deviceset="+3V3" device=""/>
+<part name="D3" library="diode" library_urn="urn:adsk.eagle:library:210" deviceset="GF1" device="" package3d_urn="urn:adsk.eagle:package:43452/2" value="1N4001"/>
+<part name="P+26" library="supply1" library_urn="urn:adsk.eagle:library:371" deviceset="+5V" device=""/>
 </parts>
 <sheets>
@@
 <wire x1="185.42" y1="114.3" x2="193.04" y2="114.3" width="0.1524" layer="91"/>
 <label x="195.58" y="114.3" size="1.778" layer="95"/>
+</segment>
+</net>
+<net name="SIG-FLOOR" class="0">
+<segment>
+<pinref part="U2" gate="A" pin="PC0"/>
+<wire x1="185.42" y1="127" x2="193.04" y2="127" width="0.1524" layer="91"/>
+<label x="195.58" y="127" size="1.778" layer="95"/>
+</segment>
+</net>
+<net name="LED-L" class="0">
+<segment>
+<wire x1="124.46" y1="88.9" x2="116.84" y2="88.9" width="0.1524" layer="91"/>
+<label x="106.68" y="88.9" size="1.778" layer="95"/>
+<pinref part="U2" gate="A" pin="PA15"/>
+</segment>
+</net>
+<net name="LED-FLOOR" class="0">
+<segment>
+<pinref part="U2" gate="A" pin="PB15"/>
+<wire x1="124.46" y1="48.26" x2="116.84" y2="48.26" width="0.1524" layer="91"/>
+<label x="101.6" y="48.26" size="1.778" layer="95"/>
+</segment>
+</net>
+<net name="LED-UI" class="0">
+<segment>
+<pinref part="U2" gate="A" pin="PB14"/>
+<wire x1="124.46" y1="50.8" x2="116.84" y2="50.8" width="0.1524" layer="91"/>
+<label x="101.6" y="50.8" size="1.778" layer="95"/>
+</segment>
+</net>
+<net name="LED-R" class="0">
+<segment>
+<pinref part="U2" gate="A" pin="PB13"/>
+<wire x1="124.46" y1="53.34" x2="116.84" y2="53.34" width="0.1524" layer="91"/>
+<label x="101.6" y="53.34" size="1.778" layer="95"/>
+</segment>
+</net>
+<net name="SW1" class="0">
+<segment>
+<pinref part="U2" gate="A" pin="PA4"/>
+<wire x1="124.46" y1="116.84" x2="116.84" y2="116.84" width="0.1524" layer="91"/>
+<label x="104.14" y="116.84" size="1.778" layer="95"/>
+</segment>
+</net>
+<net name="SW2" class="0">
+<segment>
+<pinref part="U2" gate="A" pin="PA5"/>
+<wire x1="124.46" y1="114.3" x2="116.84" y2="114.3" width="0.1524" layer="91"/>
+<label x="104.14" y="114.3" size="1.778" layer="95"/>
+</segment>
+</net>
+<net name="TOGGLE" class="0">
+<segment>
+<pinref part="U2" gate="A" pin="PA6"/>
+<wire x1="124.46" y1="111.76" x2="116.84" y2="111.76" width="0.1524" layer="91"/>
+<label x="104.14" y="111.76" size="1.778" layer="95"/>
 </segment>
 </net>
@@
 <attribute name="VALUE" x="142.24" y="71.12" size="1.778" layer="96"/>
 </instance>
+<instance part="D3" gate="D" x="248.92" y="168.91" smashed="yes" rot="R180">
+<attribute name="NAME" x="246.38" y="165.1" size="1.778" layer="95"/>
+<attribute name="VALUE" x="251.46" y="165.1" size="1.778" layer="96"/>
+</instance>
+<instance part="P+26" gate="1" x="259.08" y="175.26" smashed="yes">
+<attribute name="VALUE" x="252.476" y="172.72" size="1.778" layer="96"/>
+</instance>
 </instances>
 <busses>
@@
 <pinref part="P+18" gate="1" pin="+5V"/>
 </segment>
+<segment>
+<pinref part="D3" gate="D" pin="A"/>
+<wire x1="251.46" y1="168.91" x2="259.08" y2="168.91" width="0.1524" layer="91"/>
+<wire x1="259.08" y1="168.91" x2="259.08" y2="172.72" width="0.1524" layer="91"/>
+<pinref part="P+26" gate="1" pin="+5V"/>
+</segment>
 </net>
 <net name="SIG-FLOOR" class="0">
@@
 </segment>
 </net>
+<net name="N$31" class="0">
+<segment>
+<pinref part="X1" gate="G$1" pin="5V"/>
+<pinref part="D3" gate="D" pin="C"/>
+<wire x1="246.38" y1="168.91" x2="237.49" y2="168.91" width="0.1524" layer="91"/>
+</segment>
+</net>
