File: 004-floorSensor/004-floorSensor.sch (EAGLE design)
At the start: 8 parts, among them T1 MYPARTS_NJL7502L, T2 MYPARTS_NJL7502L, T3 MYPARTS_NJL7502L, T4 MYPARTS_NJL7502L, X1 B4B-ZR

Commit message: #WeLoveSTM32
Other:
- moved on the sheet: T1, T2, T3, T4, X1-1, X1-2, X1-3, X1-4
